File: PCB/IOlinesManagement/IO_0116.kicad_sch (KiCad schematic)
At the start: 144 parts, among them Q17 BC337, Q18 BC337, Q19 BC337, Q20 BC337, Q21 BC337, Q22 BC337, Q23 BC337, Q24 BC337, Q25 BC337, Q26 BC337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

Commit message: Duplicated components names fixed
Parts:
- renumbered C2 to C1, C1 to C2, C5 to C4, C4 to C5, Q8 to Q17, Q17 to Q18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
