File: PCB/IOlinesManagement/inputs_0116.kicad_sch (KiCad schematic)
At the start: 96 parts, among them Q25 BC327, Q34 BC327, Q51 BC327, Q52 BC327, Q53 BC327, Q54 BC327, Q55 BC327, Q56 BC327, Q57 BC327, Q58 BC327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

Commit message: fixes
Parts:
- added R17: 1K, Resistor_SMD:R_1206_3216Metric, symbol Device:R
- R143: footprint Resistor_SMD:R_1206_3216Metric -> (none)
Connections:
- net +5V: now also R17.2
- net at Q59.3 (E): now also R17.1
Changed lines of the file:
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@@
 			)
 		)
-		(property "Footprint" "Resistor_SMD:R_1206_3216Metric"
+		(property "Footprint" ""
 			(at 170.434 60.452 90)
 			(effects
@@
 					(unit 1)
 				)
+			)
+		)
+	)
+	(symbol
+		(lib_id "Device:R")
+		(at 114.554 66.802 90)
+		(unit 1)
+		(exclude_from_sim no)
+		(in_bom yes)
+		(on_board yes)
+		(dnp no)
+		(property "Reference" "R17"
+			(at 114.554 73.406 90)
+			(effects
+				(font
+					(size 1.27 1.27)
+				)
+				(hide yes)
+			)
+		)
+		(property "Value" "1K"
+			(at 114.554 66.802 90)
+			(effects
+				(font
+					(size 1.27 1.27)
+				)
+			)
+		)
+		(property "Footprint" "Resistor_SMD:R_1206_3216Metric"
+			(at 114.554 68.58 90)
+			(effects
+				(font
+					(size 1.27 1.27)
+				)
+				(hide yes)
+			)
+		)
+		(property "Datasheet" "~"
+			(at 114.554 66.802 0)
+			(effects
+				(font
+					(size 1.27 1.27)
+				)
+				(hide yes)
+			)
+		)
+		(property "Description" "Resistor"
+			(at 114.554 66.802 0)
+			(effects
+				(font
+					(size 1.27 1.27)
+				)
+				(hide yes)
+			)
+		)
+		(pin "1"
+		)
+		(pin "2"
+		)
+		(instances
+			(project "main"
+				(path "/e1cfbeff-02ed-44cc-ae25-dce7e255cb28/af0c9688-8424-44b6-99df-696fe62a0ea5"
+					(reference "R17")
+					(unit 1)
+				)

Commit message: Small fix: unused lost resistor removed
Parts:
- removed R143: 1K, symbol Device:R
Changed lines of the file:
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@@
-	(symbol
-		(lib_id "Device:R")
-		(at 170.434 58.674 90)
-		(unit 1)
-		(exclude_from_sim no)
-		(in_bom yes)
-		(on_board yes)
-		(dnp no)
-		(property "Reference" "R143"
-			(at 170.434 65.278 90)
-			(effects
-				(font
-					(size 1.27 1.27)
-				)
-				(hide yes)
-			)
-		)
-		(property "Value" "1K"
-			(at 170.434 58.674 90)
-			(effects
-				(font
-					(size 1.27 1.27)
-				)
-			)
-		)
-		(property "Footprint" ""
-			(at 170.434 60.452 90)
-			(effects
-				(font
-					(size 1.27 1.27)
-				)
-				(hide yes)
-			)
-		)
-		(property "Datasheet" "~"
-			(at 170.434 58.674 0)
-			(effects
-				(font
-					(size 1.27 1.27)
-				)
-				(hide yes)
-			)
-		)
-		(property "Description" "Resistor"
-			(at 170.434 58.674 0)
-			(effects
-				(font
-					(size 1.27 1.27)
-				)
-				(hide yes)
-			)
-		)
-		(pin "1"
-		)
-		(pin "2"
-		)
-		(instances
-			(project "main"
-				(path "/e1cfbeff-02ed-44cc-ae25-dce7e255cb28/af0c9688-8424-44b6-99df-696fe62a0ea5"
-					(reference "R143")
-					(unit 1)
-				)
-			)
-		)
-	)
 	(symbol
 		(lib_id "Device:R")
