File: PCB/IOlinesManagement/outputs_0116.kicad_sch (KiCad schematic)
At the start: 9 parts, among them J1 Conn_01x02, U1 MIC4427, U2 MIC4427, U3 MIC4427, U4 MIC4427, U5 MIC4427, U6 MIC4427, U7 MIC4427, U8 MIC4427

Commit message: Wrong electric power connection fixed
Connections:
- net GND: now reaches J1.1 (Pin_1), U1.3 (GND), U2.3 (GND), U3.3 (GND), U4.3 (GND), U5.3 (GND), U6.3 (GND), U7.3 (GND), U8.3 (GND)
- net +5V: now reaches J1.2 (Pin_2), U1.6 (V+), U2.6 (V+), U3.6 (V+), U4.6 (V+), U5.6 (V+), U6.6 (V+), U7.6 (V+), U8.6 (V+)
Changed lines of the file:
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@@
+	)
+	(junction
+		(at 165.608 141.224)
+		(diameter 0)
+		(color 0 0 0 0)
 	)
 	(junction
@@
 	(wire
 		(pts
-			(xy 143.002 141.224) (xy 185.42 141.224)
+			(xy 143.002 141.224) (xy 165.608 141.224)
 		)
 		(stroke
@@
 		(pts
 			(xy 143.002 82.296) (xy 143.002 112.776)
+		)
+		(stroke
+			(width 0)
+			(type default)
+		)
+	)
+	(wire
+		(pts
+			(xy 165.608 141.224) (xy 185.42 141.224)
 		)
 		(stroke
@@
 	)
 	(symbol
+		(lib_id "power:+5V")
+		(at 138.176 33.02 0)
+		(unit 1)
+		(exclude_from_sim no)
+		(in_bom yes)
+		(on_board yes)
+		(dnp no)
+		(property "Reference" "#PWR07"
+			(at 138.176 36.83 0)
+			(effects
+				(font
+					(size 1.27 1.27)
+				)
+				(hide yes)
+			)
+		)
+		(property "Value" "+5V"
+			(at 140.716 30.734 0)
+			(effects
+				(font
+					(size 1.27 1.27)
+				)
+			)
+		)
+		(property "Footprint" ""
+			(at 138.176 33.02 0)
+			(effects
+				(font
+					(size 1.27 1.27)
+				)
+				(hide yes)
+			)
+		)
+		(property "Datasheet" ""
+			(at 138.176 33.02 0)
+			(effects
+				(font
+					(size 1.27 1.27)
+				)
+				(hide yes)
+			)
+		)
+		(property "Description" "Power symbol creates a global label with name \"+5V\""
+			(at 138.176 33.02 0)
+			(effects
+				(font
+					(size 1.27 1.27)
+				)
+				(hide yes)
+			)
+		)
+		(pin "1"
+		)
+		(instances
+			(project "main"
+				(path "/e1cfbeff-02ed-44cc-ae25-dce7e255cb28/8998d3fd-5041-4adb-a71a-54aa0c585421"
+					(reference "#PWR07")
+					(unit 1)
+				)
+			)
+		)
+	)
+	(symbol
+		(lib_id "power:GND")
+		(at 165.608 141.224 0)
+		(unit 1)
+		(exclude_from_sim no)
+		(in_bom yes)
+		(on_board yes)
+		(dnp no)
+		(fields_autoplaced yes)
+		(property "Reference" "#PWR08"
+			(at 165.608 147.574 0)
+			(effects
+				(font
+					(size 1.27 1.27)
+				)
+				(hide yes)
+			)
+		)
+		(property "Value" "GND"
+			(at 165.608 146.05 0)
+			(effects
+				(font
+					(size 1.27 1.27)
+				)
+			)
+		)
+		(property "Footprint" ""
+			(at 165.608 141.224 0)
+			(effects
+				(font
+					(size 1.27 1.27)
+				)
+				(hide yes)
+			)
+		)
+		(property "Datasheet" ""
+			(at 165.608 141.224 0)
+			(effects
+				(font
+					(size 1.27 1.27)
+				)
+				(hide yes)
+			)
+		)
+		(property "Description" "Power symbol creates a global label with name \"GND\" , ground"
+			(at 165.608 141.224 0)
+			(effects
+				(font
+					(size 1.27 1.27)
+				)
+				(hide yes)
+			)
+		)
+		(pin "1"
+		)
+		(instances
+			(project "main"
+				(path "/e1cfbeff-02ed-44cc-ae25-dce7e255cb28/8998d3fd-5041-4adb-a71a-54aa0c585421"
+					(reference "#PWR08")
+					(unit 1)
+				)
+			)
+		)
+	)
+	(symbol
 		(lib_id "Connector_Generic:Conn_01x02")
 		(at 143.002 150.368 270)
@@
 		)
 		(instances
-			(project ""
+			(project "main"
 				(path "/e1cfbeff-02ed-44cc-ae25-dce7e255cb28/8998d3fd-5041-4adb-a71a-54aa0c585421"
 					(reference "J1")
