File: PCB/ElectricProtections/fuses.kicad_sch (KiCad schematic)
At the start: 84 parts, among them U1 CD4030BE, U2 CD4030BE, U3 CD4030BE, U4 CD4030BE

Commit message: Fixes
Parts:
- D1, D10, D11, D12, D13, D14, D15, D16, D17, D18, D19, D2, D20, D21, D22, D23, D24, D25, D26, D27, D28, D29, D3, D30, D31, D32, D4, D5, D6, D7, D8, D9: value D_Zener -> 5V; footprint (none) -> Diode_SMD:D_1206_3216Metric
- R1, R10, R11, R12, R13, R14, R15, R16, R17, R18, R19, R2, R20, R21, R22, R23, R24, R25, R26, R27, R28, R29, R3, R30, R31, R32, R4, R5, R6, R7, R8, R9: footprint (none) -> Resistor_SMD:R_1206_3216Metric
- U1, U2, U3, U4: footprint CD4030BE:DIP794W45P254L1969H508Q14 -> Package_DIP:DIP-14_W7.62mm_LongPads
