File: PCB/MasterControlUnit/inputDataStorage.kicad_sch (KiCad schematic)
At the start: 0 parts

Commit message: Under development ver
inputDataStorage.kicad_sch will be renamed to dataStorages.kicad_sch
Parts:
- added U10, U11, U12, U2, U3, U4, U6, U7, U8, U9: APS6404L-3SQR-SN, APS6404L-3SQR-SN_APY, symbol APS6404L-3SQR-SN:APS6404L-3SQR-SN
- added U5: LD1117S33TR_SOT223, Package_TO_SOT_SMD:SOT-223-3_TabPin2, symbol Regulator_Linear:LD1117S33TR_SOT223
Connections:
- new net: U2.8 (VDD), U3.8 (VDD)
- new net +3.3V: U10.8 (VDD), U11.8 (VDD), U12.8 (VDD), U4.8 (VDD), U5.2 (VO), U6.8 (VDD), U8.8 (VDD), U9.8 (VDD)
- new net +5V: U5.3 (VI)
- new net CS-B1 to ISRAM: U3.1 (/CE)
- new net CS-B2 to ISRAM: U2.1 (/CE)
- new net GND: U10.4 (VSS), U11.4 (VSS), U12.4 (VSS), U2.4 (VSS), U3.4 (VSS), U4.4 (VSS), U5.1 (GND), U6.4 (VSS), U7.4 (VSS), U8.4 (VSS), U9.4 (VSS)
- new net MISO from ISRAM: U2.2 (SO/SIO[1]), U3.2 (SO/SIO[1])
- new net MISO from OSRAM: U10.5 (SI/SIO[0]), U11.5 (SI/SIO[0]), U12.5 (SI/SIO[0]), U4.5 (SI/SIO[0]), U6.5 (SI/SIO[0]), U7.5 (SI/SIO[0]), U8.5 (SI/SIO[0]), U9.5 (SI/SIO[0])
- new net MOSI to ISRAM: U2.5 (SI/SIO[0]), U3.5 (SI/SIO[0])
- new net MOSI to OSRAM: U10.2 (SO/SIO[1]), U11.2 (SO/SIO[1]), U12.2 (SO/SIO[1]), U4.2 (SO/SIO[1]), U6.2 (SO/SIO[1]), U7.2 (SO/SIO[1]), U8.2 (SO/SIO[1])
- new net SCL/SCK to ISRAM: U2.6 (SCLK), U3.6 (SCLK)
- new net SCL/SCK to OSRAM: U10.6 (SCLK), U11.6 (SCLK), U12.6 (SCLK), U4.6 (SCLK), U6.6 (SCLK), U7.6 (SCLK), U8.6 (SCLK), U9.6 (SCLK)
- no-connect marks 0 -> 20
Other:
- company: (none) -> Panico soft
- title: (none) -> SRAM storages for test's conf/data
